File: hardware/PCB/pcb.kicad_pcb (KiCad board)
At the start: 2 copper layers, 28.5 x 108.5 mm, 14 parts, among them J1 AudioJack1, J2 AudioJack2, J3 AudioJack3, J4 AudioJack3, J5 Conn_01x06_Female, J6 Conn_01x06_Female, J7 Conn_02x05_Counter_Clockwise, J8 Conn_01x10_Male, J9 Conn_01x10_Male, U1 LM7805_TO220

Commit message: Add latest KICAD updates.
Parts:
- added ?: , , F.Cu at (130.5, 109.8)
- added ?: , , F.Cu at (130.5, 96.5)
- added C3: C1uF, Capacitor_THT:CP_Radial_D5.0mm_P2.50mm, F.Cu at (121.1, 62.5)
- added D3: LED, LED_THT:LED_D3.0mm, B.Cu at (132.2, 83.6)
- added D4: 1N4007, Diode_THT:D_DO-41_SOD81_P10.16mm_Horizontal, F.Cu at (142.4, 56.4)
- added D5: LED, LED_THT:LED_D3.0mm, B.Cu at (127.1, 78.5)
- added D6: LED, LED_THT:LED_D3.0mm, B.Cu at (127.1, 83.6)
- added D7: 1N4007, Diode_THT:D_DO-41_SOD81_P10.16mm_Horizontal, F.Cu at (138.7, 56.4)
- added R1: R, Resistor_THT:R_Axial_DIN0204_L3.6mm_D1.6mm_P2.54mm_Vertical, F.Cu at (139.8, 81.0)
- added R2: R, Resistor_THT:R_Axial_DIN0204_L3.6mm_D1.6mm_P2.54mm_Vertical, F.Cu at (139.8, 86.1)
- added R3: R, Resistor_THT:R_Axial_DIN0204_L3.6mm_D1.6mm_P2.54mm_Vertical, F.Cu at (139.8, 91.2)
- added R4: R, Resistor_THT:R_Axial_DIN0204_L3.6mm_D1.6mm_P2.54mm_Vertical, F.Cu at (139.8, 96.3)
- C1: value C100nF -> C0.1uF
- C2: value C1uF -> C100nF; footprint Capacitor_THT:CP_Radial_D5.0mm_P2.50mm -> Capacitor_THT:C_Rect_L4.0mm_W2.5mm_P2.50mm
- D1: value 1N4007 -> NeoPixel_THT; footprint Diode_THT:D_DO-41_SOD81_P10.16mm_Horizontal -> LED_THT:LED_D5.0mm-4_RGB_Staggered_Pins
- D2: value 1N4007 -> LED; footprint Diode_THT:D_DO-41_SOD81_P10.16mm_Horizontal -> LED_THT:LED_D3.0mm; moved to B.Cu
- J1: value AudioJack1 -> AudioJack3
- J2: value AudioJack2 -> AudioJack3
- J7: value Conn_02x05_Counter_Clockwise -> Conn_01x10_Male; footprint Connector_IDC:IDC-Header_2x05_P2.54mm_Vertical -> Connector_PinSocket_2.54mm:PinSocket_1x10_P2.54mm_Vertical
- J9: value Conn_01x10_Male -> Conn_02x05_Counter_Clockwise; footprint Connector_PinSocket_2.54mm:PinSocket_1x10_P2.54mm_Vertical -> Connector_IDC:IDC-Header_2x05_P2.54mm_Vertical
- moved D1 48.9 mm to (116.8, 108.8)
- moved J7 48.4 mm to (122.0, 97.9), turned to 180 degrees
- moved J5 46.1 mm to (137.3, 116.5), turned to -90 degrees
- moved J9 40.2 mm to (124.6, 49.5), turned to 90 degrees
- moved J6 36.7 mm to (137.3, 103.8), turned to -90 degrees
- moved D2 21.6 mm to (132.2, 78.5), turned to 90 degrees
- moved J8 14.5 mm to (137.3, 75.1)
- moved C1 14.0 mm to (124.1, 64.1)
- moved U1 11.2 mm to (132.7, 66.0), turned to 90 degrees
- moved C2 3.54 mm to (121.8, 57.8)
- moved J3 1.40 mm to (137.3, 138.2)
- moved J4 1.40 mm to (122.0, 138.2)
- moved J1 1.40 mm to (137.3, 120.6)
- moved J2 1.40 mm to (122.0, 120.6)
Connections:
- C1 pad 1: Net-(C1-Pad1) -> Net-(C2-Pad1)
- C1 pad 2: Net-(C1-Pad2) -> Net-(C2-Pad1)
- C2 pad 2: Net-(C1-Pad1) -> Net-(C2-Pad2)
- D1 pad 1: Net-(C2-Pad1) -> unconnected-(D1-Pad1)
- D1 pad 2: Net-(C1-Pad2) -> Net-(C2-Pad1)
- J1 pad T: Net-(J1-PadT) -> Net-(J5-Pad6)
- J2 pad T: Net-(J1-PadT) -> Net-(J5-Pad6)
- J3 pad T: Net-(J1-PadT) -> Net-(J5-Pad6)
- J4 pad T: Net-(J1-PadT) -> Net-(J5-Pad6)
- J5 pad 1: Net-(J1-PadT) -> unconnected-(J5-Pad1)
- J5 pad 6: unconnected-(J5-Pad6) -> Net-(J5-Pad6)
- J6 pad 1: Net-(C1-Pad2) -> Net-(C2-Pad2)
- J6 pad 2: Net-(C1-Pad1) -> Net-(C2-Pad1)
- J7 pad 1: Net-(D2-Pad2) -> unconnected-(J7-Pad1)
- J7 pad 10: unconnected-(J7-Pad10) -> Net-(D1-Pad4)
- J7 pad 5: unconnected-(J7-Pad5) -> Net-(J6-Pad4)
- J7 pad 6: unconnected-(J7-Pad6) -> Net-(J6-Pad3)
- J7 pad 9: Net-(C1-Pad1) -> unconnected-(J7-Pad9)
- J8 pad 2: unconnected-(J8-Pad2) -> Net-(C2-Pad1)
- J8 pad 3: unconnected-(J8-Pad3) -> Net-(C2-Pad2)
- J8 pad 5: Net-(J6-Pad4) -> Net-(J8-Pad5)
- J8 pad 6: Net-(J6-Pad3) -> Net-(J8-Pad6)
- J8 pad 7: unconnected-(J8-Pad7) -> Net-(J8-Pad7)
- J8 pad 8: unconnected-(J8-Pad8) -> Net-(J8-Pad8)
- J9 pad 1: unconnected-(J9-Pad1) -> Net-(D7-Pad2)
- J9 pad 2: Net-(C1-Pad1) -> unconnected-(J9-Pad2)
- J9 pad 3: Net-(C1-Pad2) -> unconnected-(J9-Pad3)
- J9 pad 9: unconnected-(J9-Pad9) -> Net-(C2-Pad1)
- U1 pad 1: Net-(C2-Pad1) -> Net-(C3-Pad1)
- U1 pad 2: Net-(C1-Pad1) -> Net-(C2-Pad1)
- U1 pad 3: Net-(C1-Pad2) -> Net-(C2-Pad2)
Routing:
- net Net-(C2-Pad1): track 0.00 -> 136.5 mm
- net Net-(J5-Pad6): track 0.00 -> 73.5 mm
- net Net-(C2-Pad2): track 0.00 -> 71.0 mm
- net Net-(D1-Pad4): track 0.00 -> 43.8 mm
- net Net-(C3-Pad1): track 0.00 -> 38.8 mm
- net Net-(D7-Pad2): track 0.00 -> 36.2 mm
- net Net-(J3-PadS): track 0.00 -> 32.8 mm
- net Net-(J4-PadS): track 0.00 -> 27.0 mm
- net Net-(J6-Pad3): track 0.00 -> 24.1 mm
- net Net-(D5-Pad2): track 0.00 -> 23.5 mm
- net Net-(D6-Pad2): track 0.00 -> 23.2 mm
- net Net-(J6-Pad4): track 0.00 -> 20.6 mm
- net Net-(J1-PadS): track 0.00 -> 17.9 mm
- net Net-(D2-Pad2): track 0.00 -> 13.9 mm
- net Net-(J2-PadS): track 0.00 -> 11.8 mm
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