File: hardware/PCB/pcb.kicad_sch (KiCad schematic)
At the start: 14 parts, among them J1 AudioJack3, J2 AudioJack3, J3 AudioJack3, J4 AudioJack3, J5 Conn_01x06_Female, J6 Conn_01x06_Female, J7 Conn_02x05_Counter_Clockwise, J8 Conn_01x10_Male, J9 Conn_01x10_Male, U1 LM7805_TO220

Commit message: Add latest KICAD updates.
Parts:
- added C1: C0.1uF, Capacitor_THT:C_Rect_L4.0mm_W2.5mm_P2.50mm, symbol Device:C
- added D1: NeoPixel_THT, LED_THT:LED_D5.0mm-4_RGB_Staggered_Pins, symbol LED:NeoPixel_THT
- added D2, D3, D5, D6: LED, LED_THT:LED_D3.0mm, symbol Device:LED
- added R1, R2, R3, R4: R, Resistor_THT:R_Axial_DIN0204_L3.6mm_D1.6mm_P2.54mm_Vertical, symbol Device:R
- renumbered C1 to C2, C2 to C3, D1 to D4, D2 to D7, J8 to J7, J9 to J8, J7 to J9
Connections:
- net at C2.1, C3.2, J6.2 (Pin_2)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: now also C1.1, C1.2, D1.2 (GND), D1.3 (VDD), D2.1 (K), D3.1 (K), D5.1 (K), D6.1 (K)
- net at J1.T, J2.T, J3.T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: now also J5.6 (Pin_6); no longer J5.1 (Pin_1)
- net at J8.5 (Pin_5): now also R1.2
- net at J8.6 (Pin_6): now also R2.2
- net at J8.7 (Pin_7): now also R3.2
- net at J8.8 (Pin_8): now also R4.2
- net at J7.10 (Pin_10): now also D1.4 (DIN)
- new net: D2.2 (A), R1.1
- new net: D3.2 (A), R2.1
- new net: D6.2 (A), R4.1
- new net: D5.2 (A), R3.1
